File: PCB/IRview/IRview.kicad_pcb (KiCad board)
At the start: 2 copper layers, 54 x 77.2 mm, 23 parts, among them J1 Conn_01x05_Pin, J2 Conn_01x08_Pin, J4 Conn_01x02_Pin, J5 Conn_01x11_Pin, SW1 SW_Push, SW2 SW_Push, SW3 SW_Push, SW4 SW_Push, SW5 SW_Push, SW6 SW_Push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

Commit message: pcb fixups and changes
Parts:
- removed C3: C, Capacitor_SMD:C_0603_1608Metric
- C1: value C -> 10uf; footprint Capacitor_SMD:C_0402_1005Metric -> Capacitor_THT:CP_Radial_D4.0mm_P2.00mm
- C2: value C -> 10uF; footprint Capacitor_SMD:C_0402_1005Metric -> Capacitor_THT:CP_Radial_D4.0mm_P2.00mm
- R1, R2, R3, R4: footprint Resistor_SMD:R_0402_1005Metric -> Resistor_THT:R_Axial_DIN0207_L6.3mm_D2.5mm_P7.62mm_Horizontal; moved to B.Cu
- moved C1 10.8 mm to (73.9, 101.8)
- moved C2 8.45 mm to (73.8, 87.1)
- moved R2 6.03 mm to (110.5, 68.0)
- moved R4 5.48 mm to (103.4, 77.8), turned to -90 degrees
- moved R3 2.61 mm to (93.3, 85.6)
- moved R1 1.58 mm to (110.3, 74.4)
Routing:
- net +5V: track 12.5 -> 32.1 mm, vias 0 -> 1
- net +3.3V: track 126.3 -> 139.4 mm, vias 2 -> 1
- net GND: track 6.28 -> 0.00 mm
- net SDA: track 21.1 -> 22.8 mm
- net SCL: track 31.4 -> 33.0 mm
- net D/C: track 62.7 -> 61.4 mm
- net Net-(U1-EN): track 38.4 -> 37.3 mm, vias 2 -> 1
- net Net-(U1-IO0): track 18.3 -> 17.3 mm
Other:
- outline, holes or cut-outs redrawn

Commit message: change esp and rewire
Parts:
- removed U1: ESP32-WROOM-32E-R2, RF_Module:ESP32-WROOM-32D
- added U4: ESP32-S3-WROOM-1, RF_Module:ESP32-S3-WROOM-1, F.Cu at (94.7, 63.6)
- moved R1 8.13 mm to (110.8, 82.5), turned to 90 degrees
- moved SW4 7.95 mm to (119.9, 68.5), turned to -90 degrees
- moved R3 7.77 mm to (101.0, 86.6), turned to 180 degrees
- moved R4 4.28 mm to (107.5, 78.9), turned to -100 degrees
Connections:
- R1 pad 1: Net-(U1-IO0) -> +3.3V
- R1 pad 2: +3.3V -> Net-(U4-IO0)
- R3 pad 1: SCL -> +3.3V
- R3 pad 2: +3.3V -> SCL
- SW4 pad 1: Net-(U1-IO0) -> GND
- SW4 pad 2: GND -> Net-(U4-IO0)
Routing:
- net D/C: track 61.4 -> 42.5 mm, vias 2 -> 3
- net Net-(U4-IO0): track 0.00 -> 18.4 mm
- net Net-(U1-IO0): track 17.3 -> 0.00 mm
- net LBO: track 42.2 -> 55.8 mm, vias 1 -> 2
- net SCL: track 33.0 -> 24.2 mm
- net RST: track 49.4 -> 56.0 mm
- net SDCS: track 54.6 -> 48.7 mm
- net SDA: track 22.8 -> 17.6 mm
- net +5V: track 32.1 -> 27.0 mm, vias 1 -> 0
- net BL: track 52.1 -> 47.6 mm, vias 2 -> 1
- net +3.3V: track 139.4 -> 135.6 mm
- net Net-(J4-Pin_1): track 30.7 -> 34.5 mm
- net Net-(J4-Pin_2): track 31.7 -> 35.3 mm
- net CS: track 47.5 -> 51.2 mm
- net BT1: track 88.2 -> 91.2 mm
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
Commit message: change screen
Parts:
- removed J5: Conn_01x11_Pin, Connector_PinHeader_2.54mm:PinHeader_1x11_P2.54mm_Vertical
- added J3: Conn_01x09_Socket, Connector_PinSocket_2.54mm:PinSocket_1x09_P2.54mm_Vertical, F.Cu at (105.3, 113.7)
Connections:
- U4 pad 19: BL -> LED
- U4 pad 31: SDCS -> unconnected-(U4-IO38-Pad31)
Routing:
- net SDCS: track 48.7 -> 0.00 mm, vias 2 -> 0
- net BL: track 47.6 -> 0.00 mm, vias 1 -> 0
- net LED: track 0.00 -> 46.7 mm, vias 0 -> 1
- net D/C: track 42.5 -> 61.1 mm, vias 3 -> 1
- net CS: track 51.2 -> 61.0 mm
- net RST: track 56.0 -> 61.5 mm, vias 1 -> 2
- net MISO: track 57.6 -> 53.3 mm, vias 1 -> 2
- net +3.3V: track 135.6 -> 138.1 mm
- net MOSI: track 57.7 -> 55.9 mm, vias 1 -> 2
- net EN: track 21.8 -> 22.5 mm
