File: PCB/IRview/IRview.kicad_sch (KiCad schematic)
At the start: 19 parts, among them J1 Conn_01x05_Pin, J2 Conn_01x08_Pin, J4 Conn_01x02_Pin, J5 Conn_01x11_Pin, SW1 SW_Push, SW2 SW_Push, SW3 SW_Push, SW4 SW_Push, SW5 SW_Push, SW6 SW_Push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

Commit message: pcb fixups and changes
Parts:
- removed C1, C2: C, Capacitor_SMD:C_0402_1005Metric, symbol Device:C
- removed C3: C, Capacitor_SMD:C_0603_1608Metric, symbol Device:C
- added C1: 10uf, Capacitor_THT:CP_Radial_D4.0mm_P2.00mm, symbol Device:C_Polarized
- added C2: 10uF, Capacitor_THT:CP_Radial_D4.0mm_P2.00mm, symbol Device:C_Polarized
- J1, J2, J4, J5, SW1, SW2, SW3, SW4, SW5, SW6: now left out of the parts list
- R1, R2, R3, R4: footprint Resistor_SMD:R_0402_1005Metric -> Resistor_THT:R_Axial_DIN0207_L6.3mm_D2.5mm_P7.62mm_Horizontal; now left out of the parts list
Connections:
- net +3.3V: now also C2.1
- net +5V: now also C1.1
- net GND: now also C1.2, C2.2

Commit message: change esp and rewire
Parts:
- removed U1: ESP32-WROOM-32E-R2, RF_Module:ESP32-WROOM-32D, symbol RF_Module:ESP32-WROOM-32E-R2
- added U4: ESP32-S3-WROOM-1, RF_Module:ESP32-S3-WROOM-1, symbol RF_Module:ESP32-S3-WROOM-1
Connections:
- net +3.3V: now also R1.1, R3.1, U4.2 (3V3); no longer R1.2, R3.2
- net BL: now also U4.19 (IO11)
- net BT1: now also U4.7 (IO7)
- net BT2: now also U4.6 (IO6)
- net BT3: now also U4.5 (IO5)
- net CS: now also U4.21 (IO13)
- net D/C: now also U4.22 (IO14)
- net GND: now also SW4.1, U4.1 (GND), U4.40 (GND), U4.41 (GND); no longer SW4.2
- net LBO: now also U4.25 (IO48)
- net MISO: now also U4.10 (IO17)
- net MOSI: now also U4.9 (IO16)
- net RST: now also U4.8 (IO15)
- net SCK: now also U4.20 (IO12)
- net SCL: now also R3.2, U4.11 (IO18); no longer R3.1
- net SDA: now also U4.23 (IO21)
- net SDCS: now also U4.31 (IO38)
- net at R2.2, SW5.2: now also U4.3 (EN)
- net at J4.1 (Pin_1): now also U4.36 (RXD0)
- net at J4.2 (Pin_2): now also U4.37 (TXD0)
- new net: R1.2, SW4.2, U4.27 (IO0)
- no-connect marks 9 -> 20
Other:
- moved on the sheet: C1, C2, J1, J2, J5, SW1, SW2, SW3, SW6, U2

Commit message: change screen
Parts:
- removed J5: Conn_01x11_Pin, Connector_PinHeader_2.54mm:PinHeader_1x11_P2.54mm_Vertical, symbol Connector:Conn_01x11_Pin
- added J3: Conn_01x09_Socket, Connector_PinSocket_2.54mm:PinSocket_1x09_P2.54mm_Vertical, symbol Connector:Conn_01x09_Socket
Connections:
- net +3.3V: now also J3.9 (Pin_9)
- net CS: now also J3.7 (Pin_7)
- net D/C: now also J3.5 (Pin_5)
- net GND: now also J3.8 (Pin_8)
- net MISO: now also J3.1 (Pin_1)
- net MOSI: now also J3.4 (Pin_4)
- net RST: now also J3.6 (Pin_6)
- net SCK: now also J3.3 (Pin_3)
- net BL renamed LED
- net LED: now also J3.2 (Pin_2)
- net SDCS: no longer names the net of U4.31 (IO38)
